Commit message: parkur simulasyonu ve urdf dosyalari birbirine baglandi sim_time_full launch olsuturdu yapisinda robot state publisheri da calistirip gazeboya plug in olarak veriyor.

File: install/ika_description/share/ika_description/urdf/base.xacro (robot description, xacro)
@@ -5,8 +5,12 @@
       <mass value="${mass}"/>
       <origin xyz="0 0 0" rpy="0 0 0"/>
-      <inertia ixx="${mass*(y*y+z*z)/12}" ixy="0" ixz="0" iyy="${mass*(x*x+z*z)/12}" iyz="0" izz="${mass*(x*x+y*y)/12}"/>
+      <inertia
+        ixx="${mass*(y*y+z*z)/12}" ixy="0" ixz="0"
+        iyy="${mass*(x*x+z*z)/12}" iyz="0"
+        izz="${mass*(x*x+y*y)/12}"/>
     </inertial>
   </xacro:macro>
   <xacro:macro name="ika_base">
+    <!-- base_footprint zemindedir. base_link şasenin merkezidir. -->
     <link name="base_footprint"/>
     <joint name="base_footprint_joint" type="fixed">
@@ -15,32 +19,80 @@
       <origin xyz="0 0 ${ground_clearance}" rpy="0 0 0"/>
     </joint>
+    <!-- Ana şase: robot_description.pdf içindeki 140 cm x 95 cm yapıya yakın ölçülendirilmiştir. -->
     <link name="base_link">
       <visual>
         <origin xyz="0 0 0" rpy="0 0 0"/>
-        <geometry><box size="${base_length} ${base_width} ${base_height}"/></geometry>
-        <material name="dark_gray"><color rgba="0.12 0.12 0.12 1"/></material>
+        <geometry>
+          <box size="${base_length} ${base_width} ${base_height}"/>
+        </geometry>
+        <material name="dark_gray">
+          <color rgba="0.10 0.10 0.10 1.0"/>
+        </material>
       </visual>
       <collision>
         <origin xyz="0 0 0" rpy="0 0 0"/>
-        <geometry><box size="${base_length} ${base_width} ${base_height}"/></geometry>
+        <geometry>
+          <box size="${base_length} ${base_width} ${base_height}"/>
+        </geometry>
       </collision>
       <xacro:box_inertial mass="42.0" x="${base_length}" y="${base_width}" z="${base_height}"/>
     </link>
-    <link name="upper_frame_link">
+    <!-- Sensörleri taşıyan üst şase/platform. Tüm kamera, lidar, gps, imu vb. bu şase üzerine bağlanır. -->
+    <link name="sensor_deck_link">
       <visual>
         <origin xyz="0 0 0" rpy="0 0 0"/>
-        <geometry><box size="1.05 0.65 0.06"/></geometry>
-        <material name="metal"><color rgba="0.45 0.45 0.45 1"/></material>
+        <geometry>
+          <box size="1.08 0.66 0.055"/>
+        </geometry>
+        <material name="sensor_deck_gray">
+          <color rgba="0.42 0.42 0.42 1.0"/>
+        </material>
       </visual>
-      <collision><geometry><box size="1.05 0.65 0.06"/></geometry></collision>
-      <xacro:box_inertial mass="4.0" x="1.05" y="0.65" z="0.06"/>
+      <collision>
+        <origin xyz="0 0 0" rpy="0 0 0"/>
+        <geometry>
+          <box size="1.08 0.66 0.055"/>
+        </geometry>
+      </collision>
+      <xacro:box_inertial mass="5.0" x="1.08" y="0.66" z="0.055"/>
     </link>
-    <joint name="upper_frame_joint" type="fixed">
+    <joint name="sensor_deck_joint" type="fixed">
       <parent link="base_link"/>
-      <child link="upper_frame_link"/>
-      <origin xyz="0 0 0.20" rpy="0 0 0"/>
+      <child link="sensor_deck_link"/>
+      <origin xyz="0 0 ${base_height/2 + 0.055/2 + 0.035}" rpy="0 0 0"/>
     </joint>
-    <gazebo reference="base_link"><material>Gazebo/DarkGrey</material></gazebo>
-    <gazebo reference="upper_frame_link"><material>Gazebo/Grey</material></gazebo>
+    <!-- Elektronik muhafaza: Jetson Nano, Arduino Mega, batarya ve sürücülerin sembolik kutusu. -->
+    <link name="electronics_box_link">
+      <visual>
+        <origin xyz="0 0 0" rpy="0 0 0"/>
+        <geometry>
+          <box size="0.42 0.32 0.12"/>
+        </geometry>
+        <material name="electronics_blue">
+          <color rgba="0.05 0.12 0.25 1.0"/>
+        </material>
+      </visual>
+      <collision>
+        <origin xyz="0 0 0" rpy="0 0 0"/>
+        <geometry>
+          <box size="0.42 0.32 0.12"/>
+        </geometry>
+      </collision>
+      <xacro:box_inertial mass="4.0" x="0.42" y="0.32" z="0.12"/>
+    </link>
+    <joint name="electronics_box_joint" type="fixed">
+      <parent link="sensor_deck_link"/>
+      <child link="electronics_box_link"/>
+      <origin xyz="-0.22 0 0.09" rpy="0 0 0"/>
+    </joint>
+    <gazebo reference="base_link">
+      <material>Gazebo/DarkGrey</material>
+    </gazebo>
+    <gazebo reference="sensor_deck_link">
+      <material>Gazebo/Grey</material>
+    </gazebo>
+    <gazebo reference="electronics_box_link">
+      <material>Gazebo/Blue</material>
+    </gazebo>
   </xacro:macro>
 </robot>

File: install/ika_description/share/ika_description/urdf/robot.urdf.xacro (robot description, xacro)
@@ -2,12 +2,15 @@
 <robot name="ika_teknofest_aventra" xmlns:xacro="http://www.ros.org/wiki/xacro">
   <xacro:property name="PI" value="3.14159265359"/>
+  <!-- Gerçek rapora yakın genel boyutlar: 1.40 m uzunluk, 0.95 m genişlik. -->
   <xacro:property name="base_length" value="1.40"/>
   <xacro:property name="base_width"  value="0.95"/>
-  <xacro:property name="base_height" value="0.22"/>
-  <xacro:property name="ground_clearance" value="0.34"/>
+  <xacro:property name="base_height" value="0.20"/>
+  <!-- base_link şase merkezidir. Bu değer şasenin yerden yüksekliğini belirler. -->
+  <xacro:property name="ground_clearance" value="0.44"/>
   <xacro:property name="wheel_radius" value="0.18"/>
   <xacro:property name="wheel_width"  value="0.12"/>
-  <xacro:property name="wheel_x" value="0.48"/>
-  <xacro:property name="wheel_y" value="0.54"/>
+  <xacro:property name="wheel_x" value="0.49"/>
+  <xacro:property name="wheel_y" value="0.55"/>
+  <xacro:arg name="controllers_file" default="$(find ika_control)/config/rover_controllers.yaml"/>
   <xacro:include filename="$(find ika_description)/urdf/base.xacro"/>
   <xacro:include filename="$(find ika_description)/urdf/wheels.xacro"/>
@@ -22,40 +25,54 @@
   <xacro:include filename="$(find ika_description)/urdf/environmental_sensor.xacro"/>
   <xacro:include filename="$(find ika_description)/urdf/laser_pointer.xacro"/>
+  <!-- Ana gövde ve üst sensör şasesi -->
   <xacro:ika_base/>
-  <xacro:ika_wheel name="front_left"  parent="base_link" x="${wheel_x}"  y="${wheel_y}" z="${wheel_radius}"/>
-  <xacro:ika_wheel name="rear_left"   parent="base_link" x="-${wheel_x}" y="${wheel_y}" z="${wheel_radius}"/>
+  <!-- 4 teker diferansiyel sürüş. Her tekerlek önce bacak taşıyıcıya, sonra hub üzerinden tekerleğe bağlanır. -->
+  <xacro:ika_wheel name="front_left"  parent="base_link" x="${wheel_x}"  y="${wheel_y}"  z="${wheel_radius}"/>
+  <xacro:ika_wheel name="rear_left"   parent="base_link" x="-${wheel_x}" y="${wheel_y}"  z="${wheel_radius}"/>
   <xacro:ika_wheel name="front_right" parent="base_link" x="${wheel_x}"  y="-${wheel_y}" z="${wheel_radius}"/>
   <xacro:ika_wheel name="rear_right"  parent="base_link" x="-${wheel_x}" y="-${wheel_y}" z="${wheel_radius}"/>
-  <xacro:front_camera parent="base_link" x="0.73" y="0.00" z="0.55" roll="0" pitch="0" yaw="0"/>
-  <xacro:rear_camera  parent="base_link" x="-0.73" y="0.00" z="0.50" roll="0" pitch="0" yaw="${PI}"/>
-  <xacro:lidar_sensor parent="base_link" x="0.10" y="0.00" z="0.74"/>
-  <xacro:imu_sensor parent="base_link" x="0.00" y="0.00" z="0.46"/>
-  <xacro:gps_sensor parent="base_link" x="-0.20" y="0.00" z="0.75"/>
-  <xacro:laser_range_sensor parent="base_link" x="0.76" y="0.00" z="0.42"/>
-  <xacro:environmental_sensor parent="base_link" x="-0.35" y="0.28" z="0.58"/>
-  <xacro:laser_pointer parent="base_link" x="0.35" y="0.00" z="0.68"/>
+  <!--
+    Tüm sensörler şase/üst platform üzerindedir.
+    Not: aim_camera lazer pan-tilt mekanizmasının ucundadır; pan-tilt mekanizması da sensor_deck_link'e sabitlenmiştir.
+  -->
+  <xacro:front_camera parent="sensor_deck_link" x="0.58" y="0.00" z="0.12" roll="0" pitch="0" yaw="0"/>
+  <xacro:rear_camera  parent="sensor_deck_link" x="-0.58" y="0.00" z="0.12" roll="0" pitch="0" yaw="${PI}"/>
+  <xacro:lidar_sensor parent="sensor_deck_link" x="0.05" y="0.00" z="0.19"/>
+  <xacro:imu_sensor parent="sensor_deck_link" x="0.00" y="0.00" z="0.055"/>
+  <xacro:gps_sensor parent="sensor_deck_link" x="-0.36" y="0.00" z="0.17"/>
+  <xacro:laser_range_sensor parent="sensor_deck_link" x="0.62" y="0.00" z="0.08"/>
+  <xacro:environmental_sensor parent="sensor_deck_link" x="-0.28" y="0.24" z="0.10"/>
+  <xacro:laser_pointer parent="sensor_deck_link" x="0.28" y="0.00" z="0.16"/>
   <xacro:aim_camera parent="tilt_link" x="0.12" y="0.00" z="0.03" roll="0" pitch="0" yaw="0"/>
+    <!-- gazebo_ros2_control plugin -->
   <gazebo>
-    <plugin name="ika_diff_drive" filename="libgazebo_ros_diff_drive.so">
-      <ros>
-        <namespace>/</namespace>
-        <remapping>cmd_vel:=cmd_vel</remapping>
-        <remapping>odom:=odom</remapping>
-      </ros>
-      <left_joint>front_left_wheel_joint</left_joint>
-      <left_joint>rear_left_wheel_joint</left_joint>
-      <right_joint>front_right_wheel_joint</right_joint>
-      <right_joint>rear_right_wheel_joint</right_joint>
-      <wheel_separation>1.08</wheel_separation>
-      <wheel_diameter>0.36</wheel_diameter>
-      <max_wheel_torque>80.0</max_wheel_torque>
-      <max_wheel_acceleration>3.0</max_wheel_acceleration>
-      <publish_odom>true</publish_odom>
-      <publish_odom_tf>true</publish_odom_tf>
-      <publish_wheel_tf>true</publish_wheel_tf>
-      <odometry_frame>odom</odometry_frame>
-      <robot_base_frame>base_link</robot_base_frame>
-      <update_rate>50</update_rate>
+    <plugin name="gazebo_ros2_control" filename="libgazebo_ros2_control.so">
+      <parameters>$(arg controllers_file)</parameters>
     </plugin>
   </gazebo>
+  <ros2_control name="ika_hw" type="system">
+    <hardware>
+      <plugin>gazebo_ros2_control/GazeboSystem</plugin>
+    </hardware>
+    <joint name="front_left_wheel_joint">
+      <command_interface name="velocity"/>
+      <state_interface name="position"/>
+      <state_interface name="velocity"/>
+    </joint>
+    <joint name="rear_left_wheel_joint">
+      <command_interface name="velocity"/>
+      <state_interface name="position"/>
+      <state_interface name="velocity"/>
+    </joint>
+    <joint name="front_right_wheel_joint">
+      <command_interface name="velocity"/>
+      <state_interface name="position"/>
+      <state_interface name="velocity"/>
+    </joint>
+    <joint name="rear_right_wheel_joint">
+      <command_interface name="velocity"/>
+      <state_interface name="position"/>
+      <state_interface name="velocity"/>
+    </joint>
+  </ros2_control>
 </robot>

File: install/ika_description/share/ika_description/urdf/wheels.xacro (robot description, xacro)
@@ -5,31 +5,116 @@
       <mass value="${mass}"/>
       <origin xyz="0 0 0" rpy="0 0 0"/>
-      <inertia ixx="${mass*(3*radius*radius+length*length)/12}" ixy="0" ixz="0" iyy="${mass*radius*radius/2}" iyz="0" izz="${mass*(3*radius*radius+length*length)/12}"/>
+      <inertia
+        ixx="${mass*(3*radius*radius+length*length)/12}" ixy="0" ixz="0"
+        iyy="${mass*radius*radius/2}" iyz="0"
+        izz="${mass*(3*radius*radius+length*length)/12}"/>
     </inertial>
   </xacro:macro>
+  <!--
+    Her teker için önce şaseden aşağı inen bir bacak/taşıyıcı kol oluşturulur.
+    Tekerlek doğrudan base_link'e değil, bu bacak ucuna bağlanır.
+  -->
   <xacro:macro name="ika_wheel" params="name parent x y z">
+    <xacro:property name="wheel_center_z" value="${-ground_clearance + z}"/>
+    <xacro:property name="leg_top_z" value="${-base_height/2}"/>
+    <xacro:property name="leg_bottom_z" value="${wheel_center_z}"/>
+    <xacro:property name="leg_length" value="${leg_top_z - leg_bottom_z}"/>
+    <xacro:property name="leg_mid_z" value="${(leg_top_z + leg_bottom_z)/2}"/>
+    <link name="${name}_leg_link">
+      <visual>
+        <origin xyz="0 0 0" rpy="0 0 0"/>
+        <geometry>
+          <box size="0.08 0.08 ${leg_length}"/>
+        </geometry>
+        <material name="leg_metal">
+          <color rgba="0.32 0.32 0.32 1.0"/>
+        </material>
+      </visual>
+      <collision>
+        <origin xyz="0 0 0" rpy="0 0 0"/>
+        <geometry>
+          <box size="0.08 0.08 ${leg_length}"/>
+        </geometry>
+      </collision>
+      <inertial>
+        <mass value="1.1"/>
+        <origin xyz="0 0 0" rpy="0 0 0"/>
+        <inertia ixx="0.01" ixy="0" ixz="0" iyy="0.01" iyz="0" izz="0.01"/>
+      </inertial>
+    </link>
+    <joint name="${name}_leg_joint" type="fixed">
+      <parent link="${parent}"/>
+      <child link="${name}_leg_link"/>
+      <origin xyz="${x} ${y} ${leg_mid_z}" rpy="0 0 0"/>
+    </joint>
+    <!-- Teker bağlantı göbeği -->
+    <link name="${name}_hub_link">
+      <visual>
+        <origin xyz="0 0 0" rpy="${PI/2} 0 0"/>
+        <geometry>
+          <cylinder radius="0.07" length="0.16"/>
+        </geometry>
+        <material name="hub_gray">
+          <color rgba="0.55 0.55 0.55 1.0"/>
+        </material>
+      </visual>
+      <collision>
+        <origin xyz="0 0 0" rpy="${PI/2} 0 0"/>
+        <geometry>
+          <cylinder radius="0.07" length="0.16"/>
+        </geometry>
+      </collision>
+      <xacro:cylinder_inertial mass="0.7" radius="0.07" length="0.16"/>
+    </link>
+    <joint name="${name}_hub_joint" type="fixed">
+      <parent link="${name}_leg_link"/>
+      <child link="${name}_hub_link"/>
+      <origin xyz="0 0 ${-leg_length/2}" rpy="0 0 0"/>
+    </joint>
     <link name="${name}_wheel_link">
       <visual>
         <origin xyz="0 0 0" rpy="${PI/2} 0 0"/>
-        <geometry><cylinder radius="${wheel_radius}" length="${wheel_width}"/></geometry>
-        <material name="rubber"><color rgba="0.02 0.02 0.02 1"/></material>
+        <geometry>
+          <cylinder radius="${wheel_radius}" length="${wheel_width}"/>
+        </geometry>
+        <material name="rubber">
+          <color rgba="0.02 0.02 0.02 1.0"/>
+        </material>
       </visual>
       <collision>
         <origin xyz="0 0 0" rpy="${PI/2} 0 0"/>
-        <geometry><cylinder radius="${wheel_radius}" length="${wheel_width}"/></geometry>
+        <geometry>
+          <cylinder radius="${wheel_radius}" length="${wheel_width}"/>
+        </geometry>
       </collision>
-      <xacro:cylinder_inertial mass="2.0" radius="${wheel_radius}" length="${wheel_width}"/>
+      <xacro:cylinder_inertial mass="2.4" radius="${wheel_radius}" length="${wheel_width}"/>
     </link>
     <joint name="${name}_wheel_joint" type="continuous">
-      <parent link="${parent}"/>
+      <parent link="${name}_hub_link"/>
       <child link="${name}_wheel_link"/>
-      <origin xyz="${x} ${y} ${-ground_clearance + z}" rpy="0 0 0"/>
+      <origin xyz="0 0 0" rpy="0 0 0"/>
       <axis xyz="0 1 0"/>
-      <dynamics damping="0.2" friction="0.1"/>
+      <dynamics damping="0.20" friction="0.10"/>
     </joint>
+    <transmission name="${name}_wheel_transmission">
+      <type>transmission_interface/SimpleTransmission</type>
+      <joint name="${name}_wheel_joint">
+        <hardwareInterface>velocity</hardwareInterface>
+      </joint>
+      <actuator name="${name}_wheel_motor">
+        <hardwareInterface>velocity</hardwareInterface>
+        <mechanicalReduction>1</mechanicalReduction>
+      </actuator>
+    </transmission>
+    <gazebo reference="${name}_leg_link">
+      <material>Gazebo/Grey</material>
+    </gazebo>
+    <gazebo reference="${name}_hub_link">
+      <material>Gazebo/Grey</material>
+    </gazebo>
     <gazebo reference="${name}_wheel_link">
       <material>Gazebo/Black</material>
-      <mu1>1.4</mu1>
-      <mu2>1.4</mu2>
+      <mu1>1.45</mu1>
+      <mu2>1.45</mu2>
       <kp>1000000</kp>
       <kd>1</kd>
