Commit message: lidar sensorleri ve 3 kamera rviz ve gazeboda calisir duruma getirildi.

File: install/ika_description/share/ika_description/urdf/base.xacro (robot description, xacro)
@@ -1,98 +1 @@
-<?xml version="1.0"?>
-<robot xmlns:xacro="http://www.ros.org/wiki/xacro">
-  <xacro:macro name="box_inertial" params="mass x y z">
-    <inertial>
-      <mass value="${mass}"/>
-      <origin xyz="0 0 0" rpy="0 0 0"/>
-      <inertia
-        ixx="${mass*(y*y+z*z)/12}" ixy="0" ixz="0"
-        iyy="${mass*(x*x+z*z)/12}" iyz="0"
-        izz="${mass*(x*x+y*y)/12}"/>
-    </inertial>
-  </xacro:macro>
-  <xacro:macro name="ika_base">
-    <!-- base_footprint zemindedir. base_link şasenin merkezidir. -->
-    <link name="base_footprint"/>
-    <joint name="base_footprint_joint" type="fixed">
-      <parent link="base_footprint"/>
-      <child link="base_link"/>
-      <origin xyz="0 0 ${ground_clearance}" rpy="0 0 0"/>
-    </joint>
-    <!-- Ana şase: robot_description.pdf içindeki 140 cm x 95 cm yapıya yakın ölçülendirilmiştir. -->
-    <link name="base_link">
-      <visual>
-        <origin xyz="0 0 0" rpy="0 0 0"/>
-        <geometry>
-          <box size="${base_length} ${base_width} ${base_height}"/>
-        </geometry>
-        <material name="dark_gray">
-          <color rgba="0.10 0.10 0.10 1.0"/>
-        </material>
-      </visual>
-      <collision>
-        <origin xyz="0 0 0" rpy="0 0 0"/>
-        <geometry>
-          <box size="${base_length} ${base_width} ${base_height}"/>
-        </geometry>
-      </collision>
-      <xacro:box_inertial mass="42.0" x="${base_length}" y="${base_width}" z="${base_height}"/>
-    </link>
-    <!-- Sensörleri taşıyan üst şase/platform. Tüm kamera, lidar, gps, imu vb. bu şase üzerine bağlanır. -->
-    <link name="sensor_deck_link">
-      <visual>
-        <origin xyz="0 0 0" rpy="0 0 0"/>
-        <geometry>
-          <box size="1.08 0.66 0.055"/>
-        </geometry>
-        <material name="sensor_deck_gray">
-          <color rgba="0.42 0.42 0.42 1.0"/>
-        </material>
-      </visual>
-      <collision>
-        <origin xyz="0 0 0" rpy="0 0 0"/>
-        <geometry>
-          <box size="1.08 0.66 0.055"/>
-        </geometry>
-      </collision>
-      <xacro:box_inertial mass="5.0" x="1.08" y="0.66" z="0.055"/>
-    </link>
-    <joint name="sensor_deck_joint" type="fixed">
-      <parent link="base_link"/>
-      <child link="sensor_deck_link"/>
-      <origin xyz="0 0 ${base_height/2 + 0.055/2 + 0.035}" rpy="0 0 0"/>
-    </joint>
-    <!-- Elektronik muhafaza: Jetson Nano, Arduino Mega, batarya ve sürücülerin sembolik kutusu. -->
-    <link name="electronics_box_link">
-      <visual>
-        <origin xyz="0 0 0" rpy="0 0 0"/>
-        <geometry>
-          <box size="0.42 0.32 0.12"/>
-        </geometry>
-        <material name="electronics_blue">
-          <color rgba="0.05 0.12 0.25 1.0"/>
-        </material>
-      </visual>
-      <collision>
-        <origin xyz="0 0 0" rpy="0 0 0"/>
-        <geometry>
-          <box size="0.42 0.32 0.12"/>
-        </geometry>
-      </collision>
-      <xacro:box_inertial mass="4.0" x="0.42" y="0.32" z="0.12"/>
-    </link>
-    <joint name="electronics_box_joint" type="fixed">
-      <parent link="sensor_deck_link"/>
-      <child link="electronics_box_link"/>
-      <origin xyz="-0.22 0 0.09" rpy="0 0 0"/>
-    </joint>
-    <gazebo reference="base_link">
-      <material>Gazebo/DarkGrey</material>
-    </gazebo>
-    <gazebo reference="sensor_deck_link">
-      <material>Gazebo/Grey</material>
-    </gazebo>
-    <gazebo reference="electronics_box_link">
-      <material>Gazebo/Blue</material>
-    </gazebo>
-  </xacro:macro>
-</robot>
+/home/sukru/ika_teknofest_aventra_ws/src/ika_description/urdf/base.xacro

File: install/ika_description/share/ika_description/urdf/camera_aim.xacro (robot description, xacro)
@@ -1,25 +1 @@
-<?xml version="1.0"?>
-<robot xmlns:xacro="http://www.ros.org/wiki/xacro">
-  <xacro:macro name="aim_camera" params="parent x y z roll pitch yaw">
-    <link name="aim_camera_link">
-      <visual><geometry><box size="0.05 0.06 0.04"/></geometry><material name="red"><color rgba="0.9 0.05 0.05 1"/></material></visual>
-      <collision><geometry><box size="0.05 0.06 0.04"/></geometry></collision>
-      <inertial><mass value="0.12"/><inertia ixx="0.00008" ixy="0" ixz="0" iyy="0.00008" iyz="0" izz="0.00008"/></inertial>
-    </link>
-    <joint name="aim_camera_joint" type="fixed">
-      <parent link="${parent}"/><child link="aim_camera_link"/>
-      <origin xyz="${x} ${y} ${z}" rpy="${roll} ${pitch} ${yaw}"/>
-    </joint>
-    <gazebo reference="aim_camera_link">
-      <sensor name="aim_camera" type="camera">
-        <update_rate>30</update_rate>
-        <camera><horizontal_fov>0.70</horizontal_fov><image><width>1280</width><height>720</height><format>R8G8B8</format></image><clip><near>0.05</near><far>40</far></clip></camera>
-        <plugin name="aim_camera_controller" filename="libgazebo_ros_camera.so">
-          <ros><namespace>/</namespace></ros>
-          <camera_name>aim_camera</camera_name>
-          <frame_name>aim_camera_link</frame_name>
-        </plugin>
-      </sensor>
-    </gazebo>
-  </xacro:macro>
-</robot>
+/home/sukru/ika_teknofest_aventra_ws/src/ika_description/urdf/camera_aim.xacro

File: install/ika_description/share/ika_description/urdf/camera_front.xacro (robot description, xacro)
@@ -1,25 +1 @@
-<?xml version="1.0"?>
-<robot xmlns:xacro="http://www.ros.org/wiki/xacro">
-  <xacro:macro name="front_camera" params="parent x y z roll pitch yaw">
-    <link name="front_camera_link">
-      <visual><geometry><box size="0.06 0.08 0.05"/></geometry><material name="blue"><color rgba="0 0.15 0.9 1"/></material></visual>
-      <collision><geometry><box size="0.06 0.08 0.05"/></geometry></collision>
-      <inertial><mass value="0.15"/><inertia ixx="0.0001" ixy="0" ixz="0" iyy="0.0001" iyz="0" izz="0.0001"/></inertial>
-    </link>
-    <joint name="front_camera_joint" type="fixed">
-      <parent link="${parent}"/><child link="front_camera_link"/>
-      <origin xyz="${x} ${y} ${z}" rpy="${roll} ${pitch} ${yaw}"/>
-    </joint>
-    <gazebo reference="front_camera_link">
-      <sensor name="front_camera" type="camera">
-        <update_rate>30</update_rate>
-        <camera><horizontal_fov>1.396</horizontal_fov><image><width>1280</width><height>720</height><format>R8G8B8</format></image><clip><near>0.05</near><far>80</far></clip></camera>
-        <plugin name="front_camera_controller" filename="libgazebo_ros_camera.so">
-          <ros><namespace>/</namespace></ros>
-          <camera_name>front_camera</camera_name>
-          <frame_name>front_camera_link</frame_name>
-        </plugin>
-      </sensor>
-    </gazebo>
-  </xacro:macro>
-</robot>
+/home/sukru/ika_teknofest_aventra_ws/src/ika_description/urdf/camera_front.xacro

File: install/ika_description/share/ika_description/urdf/camera_rear.xacro (robot description, xacro)
@@ -1,25 +1 @@
-<?xml version="1.0"?>
-<robot xmlns:xacro="http://www.ros.org/wiki/xacro">
-  <xacro:macro name="rear_camera" params="parent x y z roll pitch yaw">
-    <link name="rear_camera_link">
-      <visual><geometry><box size="0.06 0.08 0.05"/></geometry><material name="green"><color rgba="0 0.7 0.1 1"/></material></visual>
-      <collision><geometry><box size="0.06 0.08 0.05"/></geometry></collision>
-      <inertial><mass value="0.15"/><inertia ixx="0.0001" ixy="0" ixz="0" iyy="0.0001" iyz="0" izz="0.0001"/></inertial>
-    </link>
-    <joint name="rear_camera_joint" type="fixed">
-      <parent link="${parent}"/><child link="rear_camera_link"/>
-      <origin xyz="${x} ${y} ${z}" rpy="${roll} ${pitch} ${yaw}"/>
-    </joint>
-    <gazebo reference="rear_camera_link">
-      <sensor name="rear_camera" type="camera">
-        <update_rate>30</update_rate>
-        <camera><horizontal_fov>1.396</horizontal_fov><image><width>1280</width><height>720</height><format>R8G8B8</format></image><clip><near>0.05</near><far>80</far></clip></camera>
-        <plugin name="rear_camera_controller" filename="libgazebo_ros_camera.so">
-          <ros><namespace>/</namespace></ros>
-          <camera_name>rear_camera</camera_name>
-          <frame_name>rear_camera_link</frame_name>
-        </plugin>
-      </sensor>
-    </gazebo>
-  </xacro:macro>
-</robot>
+/home/sukru/ika_teknofest_aventra_ws/src/ika_description/urdf/camera_rear.xacro

File: install/ika_description/share/ika_description/urdf/encoder.xacro (robot description, xacro)
@@ -1,4 +1 @@
-<?xml version="1.0"?>
-<robot xmlns:xacro="http://www.ros.org/wiki/xacro">
-  <!-- Enkoderler fiziksel robotta teker motor millerinde olur. Simülasyonda wheel_joint state ve diff_drive /odom bu görevi görür. -->
-</robot>
+/home/sukru/ika_teknofest_aventra_ws/src/ika_description/urdf/encoder.xacro

File: install/ika_description/share/ika_description/urdf/environmental_sensor.xacro (robot description, xacro)
@@ -1,12 +1 @@
-<?xml version="1.0"?>
-<robot xmlns:xacro="http://www.ros.org/wiki/xacro">
-  <xacro:macro name="environmental_sensor" params="parent x y z">
-    <link name="environmental_sensor_link">
-      <visual><geometry><box size="0.05 0.05 0.03"/></geometry><material name="cyan"><color rgba="0 0.8 0.9 1"/></material></visual>
-      <collision><geometry><box size="0.05 0.05 0.03"/></geometry></collision>
-      <inertial><mass value="0.04"/><inertia ixx="0.00001" ixy="0" ixz="0" iyy="0.00001" iyz="0" izz="0.00001"/></inertial>
-    </link>
-    <joint name="environmental_sensor_joint" type="fixed"><parent link="${parent}"/><child link="environmental_sensor_link"/><origin xyz="${x} ${y} ${z}" rpy="0 0 0"/></joint>
-    <!-- Gazebo Classic içinde BME280 için standart hazır plugin yok. Bu link gerçek/sim çevre node'unun frame'i olarak kullanılır. -->
-  </xacro:macro>
-</robot>
+/home/sukru/ika_teknofest_aventra_ws/src/ika_description/urdf/environmental_sensor.xacro

File: install/ika_description/share/ika_description/urdf/gps.xacro (robot description, xacro)
@@ -1,16 +1 @@
-<?xml version="1.0"?>
-<robot xmlns:xacro="http://www.ros.org/wiki/xacro">
-  <xacro:macro name="gps_sensor" params="parent x y z">
-    <link name="gps_link"><visual><geometry><box size="0.08 0.08 0.03"/></geometry><material name="white"><color rgba="0.9 0.9 0.9 1"/></material></visual><collision><geometry><box size="0.08 0.08 0.03"/></geometry></collision><inertial><mass value="0.08"/><inertia ixx="0.00002" ixy="0" ixz="0" iyy="0.00002" iyz="0" izz="0.00002"/></inertial></link>
-    <joint name="gps_joint" type="fixed"><parent link="${parent}"/><child link="gps_link"/><origin xyz="${x} ${y} ${z}" rpy="0 0 0"/></joint>
-    <gazebo reference="gps_link">
-      <sensor name="gps" type="gps">
-        <update_rate>5</update_rate>
-        <plugin name="gps_controller" filename="libgazebo_ros_gps_sensor.so">
-          <ros><remapping>~/out:=gps/fix</remapping></ros>
-          <frame_name>gps_link</frame_name>
-        </plugin>
-      </sensor>
-    </gazebo>
-  </xacro:macro>
-</robot>
+/home/sukru/ika_teknofest_aventra_ws/src/ika_description/urdf/gps.xacro

File: install/ika_description/share/ika_description/urdf/imu.xacro (robot description, xacro)
@@ -1,16 +1 @@
-<?xml version="1.0"?>
-<robot xmlns:xacro="http://www.ros.org/wiki/xacro">
-  <xacro:macro name="imu_sensor" params="parent x y z">
-    <link name="imu_link"><visual><geometry><box size="0.05 0.04 0.02"/></geometry><material name="orange"><color rgba="1 0.45 0 1"/></material></visual><collision><geometry><box size="0.05 0.04 0.02"/></geometry></collision><inertial><mass value="0.05"/><inertia ixx="0.00001" ixy="0" ixz="0" iyy="0.00001" iyz="0" izz="0.00001"/></inertial></link>
-    <joint name="imu_joint" type="fixed"><parent link="${parent}"/><child link="imu_link"/><origin xyz="${x} ${y} ${z}" rpy="0 0 0"/></joint>
-    <gazebo reference="imu_link">
-      <sensor name="imu_sensor" type="imu">
-        <update_rate>100</update_rate>
-        <plugin name="imu_controller" filename="libgazebo_ros_imu_sensor.so">
-          <ros><remapping>~/out:=imu/data</remapping></ros>
-          <frame_name>imu_link</frame_name>
-        </plugin>
-      </sensor>
-    </gazebo>
-  </xacro:macro>
-</robot>
+/home/sukru/ika_teknofest_aventra_ws/src/ika_description/urdf/imu.xacro

File: install/ika_description/share/ika_description/urdf/laser_pointer.xacro (robot description, xacro)
@@ -1,13 +1 @@
-<?xml version="1.0"?>
-<robot xmlns:xacro="http://www.ros.org/wiki/xacro">
-  <xacro:macro name="laser_pointer" params="parent x y z">
-    <link name="pan_base_link"><visual><geometry><cylinder radius="0.07" length="0.04"/></geometry><material name="black"><color rgba="0 0 0 1"/></material></visual><collision><geometry><cylinder radius="0.07" length="0.04"/></geometry></collision><inertial><mass value="0.3"/><inertia ixx="0.0002" ixy="0" ixz="0" iyy="0.0002" iyz="0" izz="0.0002"/></inertial></link>
-    <joint name="pan_base_joint" type="fixed"><parent link="${parent}"/><child link="pan_base_link"/><origin xyz="${x} ${y} ${z}" rpy="0 0 0"/></joint>
-    <link name="pan_link"><visual><geometry><box size="0.12 0.08 0.08"/></geometry><material name="gray"><color rgba="0.5 0.5 0.5 1"/></material></visual><collision><geometry><box size="0.12 0.08 0.08"/></geometry></collision><inertial><mass value="0.25"/><inertia ixx="0.0002" ixy="0" ixz="0" iyy="0.0002" iyz="0" izz="0.0002"/></inertial></link>
-    <joint name="pan_joint" type="revolute"><parent link="pan_base_link"/><child link="pan_link"/><origin xyz="0 0 0.05" rpy="0 0 0"/><axis xyz="0 0 1"/><limit lower="-1.57" upper="1.57" effort="8" velocity="1.5"/><dynamics damping="0.05" friction="0.02"/></joint>
-    <link name="tilt_link"><visual><geometry><box size="0.18 0.05 0.05"/></geometry><material name="red"><color rgba="0.9 0 0 1"/></material></visual><collision><geometry><box size="0.18 0.05 0.05"/></geometry></collision><inertial><mass value="0.20"/><inertia ixx="0.00015" ixy="0" ixz="0" iyy="0.00015" iyz="0" izz="0.00015"/></inertial></link>
-    <joint name="tilt_joint" type="revolute"><parent link="pan_link"/><child link="tilt_link"/><origin xyz="0.06 0 0" rpy="0 0 0"/><axis xyz="0 1 0"/><limit lower="-0.8" upper="0.8" effort="8" velocity="1.5"/><dynamics damping="0.05" friction="0.02"/></joint>
-    <link name="laser_pointer_link"><visual><origin xyz="0.08 0 0" rpy="0 1.5708 0"/><geometry><cylinder radius="0.012" length="0.16"/></geometry><material name="laser_red"><color rgba="1 0 0 1"/></material></visual><collision><origin xyz="0.08 0 0" rpy="0 1.5708 0"/><geometry><cylinder radius="0.012" length="0.16"/></geometry></collision><inertial><mass value="0.06"/><inertia ixx="0.00001" ixy="0" ixz="0" iyy="0.00001" iyz="0" izz="0.00001"/></inertial></link>
-    <joint name="laser_pointer_joint" type="fixed"><parent link="tilt_link"/><child link="laser_pointer_link"/><origin xyz="0.12 0 0" rpy="0 0 0"/></joint>
-  </xacro:macro>
-</robot>
+/home/sukru/ika_teknofest_aventra_ws/src/ika_description/urdf/laser_pointer.xacro

File: install/ika_description/share/ika_description/urdf/laser_range.xacro (robot description, xacro)
@@ -1,19 +1 @@
-<?xml version="1.0"?>
-<robot xmlns:xacro="http://www.ros.org/wiki/xacro">
-  <xacro:macro name="laser_range_sensor" params="parent x y z">
-    <link name="laser_range_link"><visual><geometry><box size="0.04 0.04 0.04"/></geometry><material name="purple"><color rgba="0.45 0 0.8 1"/></material></visual><collision><geometry><box size="0.04 0.04 0.04"/></geometry></collision><inertial><mass value="0.04"/><inertia ixx="0.00001" ixy="0" ixz="0" iyy="0.00001" iyz="0" izz="0.00001"/></inertial></link>
-    <joint name="laser_range_joint" type="fixed"><parent link="${parent}"/><child link="laser_range_link"/><origin xyz="${x} ${y} ${z}" rpy="0 0 0"/></joint>
-    <gazebo reference="laser_range_link">
-      <sensor name="front_tof" type="ray">
-        <update_rate>20</update_rate>
-        <ray><scan><horizontal><samples>1</samples><resolution>1</resolution><min_angle>0</min_angle><max_angle>0</max_angle></horizontal></scan><range><min>0.04</min><max>4.0</max><resolution>0.005</resolution></range></ray>
-        <plugin name="front_range_controller" filename="libgazebo_ros_ray_sensor.so">
-          <ros><remapping>~/out:=range/front</remapping></ros>
-          <output_type>sensor_msgs/Range</output_type>
-          <frame_name>laser_range_link</frame_name>
-          <radiation_type>infrared</radiation_type>
-        </plugin>
-      </sensor>
-    </gazebo>
-  </xacro:macro>
-</robot>
+/home/sukru/ika_teknofest_aventra_ws/src/ika_description/urdf/laser_range.xacro

File: install/ika_description/share/ika_description/urdf/lidar.xacro (robot description, xacro)
@@ -1,22 +1 @@
-<?xml version="1.0"?>
-<robot xmlns:xacro="http://www.ros.org/wiki/xacro">
-  <xacro:macro name="lidar_sensor" params="parent x y z">
-    <link name="lidar_link">
-      <visual><geometry><cylinder radius="0.06" length="0.05"/></geometry><material name="black"><color rgba="0 0 0 1"/></material></visual>
-      <collision><geometry><cylinder radius="0.06" length="0.05"/></geometry></collision>
-      <inertial><mass value="0.25"/><inertia ixx="0.0003" ixy="0" ixz="0" iyy="0.0003" iyz="0" izz="0.0003"/></inertial>
-    </link>
-    <joint name="lidar_joint" type="fixed"><parent link="${parent}"/><child link="lidar_link"/><origin xyz="${x} ${y} ${z}" rpy="0 0 0"/></joint>
-    <gazebo reference="lidar_link">
-      <sensor name="lidar" type="ray">
-        <update_rate>10</update_rate>
-        <ray><scan><horizontal><samples>720</samples><resolution>1</resolution><min_angle>-3.14159</min_angle><max_angle>3.14159</max_angle></horizontal></scan><range><min>0.12</min><max>12.0</max><resolution>0.01</resolution></range></ray>
-        <plugin name="lidar_controller" filename="libgazebo_ros_ray_sensor.so">
-          <ros><remapping>~/out:=scan</remapping></ros>
-          <output_type>sensor_msgs/LaserScan</output_type>
-          <frame_name>lidar_link</frame_name>
-        </plugin>
-      </sensor>
-    </gazebo>
-  </xacro:macro>
-</robot>
+/home/sukru/ika_teknofest_aventra_ws/src/ika_description/urdf/lidar.xacro

File: install/ika_description/share/ika_description/urdf/robot.urdf.xacro (robot description, xacro)
@@ -1,78 +1 @@
-<?xml version="1.0"?>
-<robot name="ika_teknofest_aventra" xmlns:xacro="http://www.ros.org/wiki/xacro">
-  <xacro:property name="PI" value="3.14159265359"/>
-  <!-- Gerçek rapora yakın genel boyutlar: 1.40 m uzunluk, 0.95 m genişlik. -->
-  <xacro:property name="base_length" value="1.40"/>
-  <xacro:property name="base_width"  value="0.95"/>
-  <xacro:property name="base_height" value="0.20"/>
-  <!-- base_link şase merkezidir. Bu değer şasenin yerden yüksekliğini belirler. -->
-  <xacro:property name="ground_clearance" value="0.44"/>
-  <xacro:property name="wheel_radius" value="0.18"/>
-  <xacro:property name="wheel_width"  value="0.12"/>
-  <xacro:property name="wheel_x" value="0.49"/>
-  <xacro:property name="wheel_y" value="0.55"/>
-  <xacro:arg name="controllers_file" default="$(find ika_control)/config/rover_controllers.yaml"/>
-  <xacro:include filename="$(find ika_description)/urdf/base.xacro"/>
-  <xacro:include filename="$(find ika_description)/urdf/wheels.xacro"/>
-  <xacro:include filename="$(find ika_description)/urdf/camera_front.xacro"/>
-  <xacro:include filename="$(find ika_description)/urdf/camera_rear.xacro"/>
-  <xacro:include filename="$(find ika_description)/urdf/camera_aim.xacro"/>
-  <xacro:include filename="$(find ika_description)/urdf/lidar.xacro"/>
-  <xacro:include filename="$(find ika_description)/urdf/imu.xacro"/>
-  <xacro:include filename="$(find ika_description)/urdf/gps.xacro"/>
-  <xacro:include filename="$(find ika_description)/urdf/encoder.xacro"/>
-  <xacro:include filename="$(find ika_description)/urdf/laser_range.xacro"/>
-  <xacro:include filename="$(find ika_description)/urdf/environmental_sensor.xacro"/>
-  <xacro:include filename="$(find ika_description)/urdf/laser_pointer.xacro"/>
-  <!-- Ana gövde ve üst sensör şasesi -->
-  <xacro:ika_base/>
-  <!-- 4 teker diferansiyel sürüş. Her tekerlek önce bacak taşıyıcıya, sonra hub üzerinden tekerleğe bağlanır. -->
-  <xacro:ika_wheel name="front_left"  parent="base_link" x="${wheel_x}"  y="${wheel_y}"  z="${wheel_radius}"/>
-  <xacro:ika_wheel name="rear_left"   parent="base_link" x="-${wheel_x}" y="${wheel_y}"  z="${wheel_radius}"/>
-  <xacro:ika_wheel name="front_right" parent="base_link" x="${wheel_x}"  y="-${wheel_y}" z="${wheel_radius}"/>
-  <xacro:ika_wheel name="rear_right"  parent="base_link" x="-${wheel_x}" y="-${wheel_y}" z="${wheel_radius}"/>
-  <!--
-    Tüm sensörler şase/üst platform üzerindedir.
-    Not: aim_camera lazer pan-tilt mekanizmasının ucundadır; pan-tilt mekanizması da sensor_deck_link'e sabitlenmiştir.
-  -->
-  <xacro:front_camera parent="sensor_deck_link" x="0.58" y="0.00" z="0.12" roll="0" pitch="0" yaw="0"/>
-  <xacro:rear_camera  parent="sensor_deck_link" x="-0.58" y="0.00" z="0.12" roll="0" pitch="0" yaw="${PI}"/>
-  <xacro:lidar_sensor parent="sensor_deck_link" x="0.05" y="0.00" z="0.19"/>
-  <xacro:imu_sensor parent="sensor_deck_link" x="0.00" y="0.00" z="0.055"/>
-  <xacro:gps_sensor parent="sensor_deck_link" x="-0.36" y="0.00" z="0.17"/>
-  <xacro:laser_range_sensor parent="sensor_deck_link" x="0.62" y="0.00" z="0.08"/>
-  <xacro:environmental_sensor parent="sensor_deck_link" x="-0.28" y="0.24" z="0.10"/>
-  <xacro:laser_pointer parent="sensor_deck_link" x="0.28" y="0.00" z="0.16"/>
-  <xacro:aim_camera parent="tilt_link" x="0.12" y="0.00" z="0.03" roll="0" pitch="0" yaw="0"/>
-    <!-- gazebo_ros2_control plugin -->
-  <gazebo>
-    <plugin name="gazebo_ros2_control" filename="libgazebo_ros2_control.so">
-      <parameters>$(arg controllers_file)</parameters>
-    </plugin>
-  </gazebo>
-  <ros2_control name="ika_hw" type="system">
-    <hardware>
-      <plugin>gazebo_ros2_control/GazeboSystem</plugin>
-    </hardware>
-    <joint name="front_left_wheel_joint">
-      <command_interface name="velocity"/>
-      <state_interface name="position"/>
-      <state_interface name="velocity"/>
-    </joint>
-    <joint name="rear_left_wheel_joint">
-      <command_interface name="velocity"/>
-      <state_interface name="position"/>
-      <state_interface name="velocity"/>
-    </joint>
-    <joint name="front_right_wheel_joint">
-      <command_interface name="velocity"/>
-      <state_interface name="position"/>
-      <state_interface name="velocity"/>
-    </joint>
-    <joint name="rear_right_wheel_joint">
-      <command_interface name="velocity"/>
-      <state_interface name="position"/>
-      <state_interface name="velocity"/>
-    </joint>
-  </ros2_control>
-</robot>
+/home/sukru/ika_teknofest_aventra_ws/src/ika_description/urdf/robot.urdf.xacro
