Commit message: lidar sensorleri ve 3 kamera rviz ve gazeboda calisir duruma getirildi.

File: install/ika_description/share/ika_description/urdf/wheels.xacro (robot description, xacro)
@@ -1,123 +1 @@
-<?xml version="1.0"?>
-<robot xmlns:xacro="http://www.ros.org/wiki/xacro">
-  <xacro:macro name="cylinder_inertial" params="mass radius length">
-    <inertial>
-      <mass value="${mass}"/>
-      <origin xyz="0 0 0" rpy="0 0 0"/>
-      <inertia
-        ixx="${mass*(3*radius*radius+length*length)/12}" ixy="0" ixz="0"
-        iyy="${mass*radius*radius/2}" iyz="0"
-        izz="${mass*(3*radius*radius+length*length)/12}"/>
-    </inertial>
-  </xacro:macro>
-  <!--
-    Her teker için önce şaseden aşağı inen bir bacak/taşıyıcı kol oluşturulur.
-    Tekerlek doğrudan base_link'e değil, bu bacak ucuna bağlanır.
-  -->
-  <xacro:macro name="ika_wheel" params="name parent x y z">
-    <xacro:property name="wheel_center_z" value="${-ground_clearance + z}"/>
-    <xacro:property name="leg_top_z" value="${-base_height/2}"/>
-    <xacro:property name="leg_bottom_z" value="${wheel_center_z}"/>
-    <xacro:property name="leg_length" value="${leg_top_z - leg_bottom_z}"/>
-    <xacro:property name="leg_mid_z" value="${(leg_top_z + leg_bottom_z)/2}"/>
-    <link name="${name}_leg_link">
-      <visual>
-        <origin xyz="0 0 0" rpy="0 0 0"/>
-        <geometry>
-          <box size="0.08 0.08 ${leg_length}"/>
-        </geometry>
-        <material name="leg_metal">
-          <color rgba="0.32 0.32 0.32 1.0"/>
-        </material>
-      </visual>
-      <collision>
-        <origin xyz="0 0 0" rpy="0 0 0"/>
-        <geometry>
-          <box size="0.08 0.08 ${leg_length}"/>
-        </geometry>
-      </collision>
-      <inertial>
-        <mass value="1.1"/>
-        <origin xyz="0 0 0" rpy="0 0 0"/>
-        <inertia ixx="0.01" ixy="0" ixz="0" iyy="0.01" iyz="0" izz="0.01"/>
-      </inertial>
-    </link>
-    <joint name="${name}_leg_joint" type="fixed">
-      <parent link="${parent}"/>
-      <child link="${name}_leg_link"/>
-      <origin xyz="${x} ${y} ${leg_mid_z}" rpy="0 0 0"/>
-    </joint>
-    <!-- Teker bağlantı göbeği -->
-    <link name="${name}_hub_link">
-      <visual>
-        <origin xyz="0 0 0" rpy="${PI/2} 0 0"/>
-        <geometry>
-          <cylinder radius="0.07" length="0.16"/>
-        </geometry>
-        <material name="hub_gray">
-          <color rgba="0.55 0.55 0.55 1.0"/>
-        </material>
-      </visual>
-      <collision>
-        <origin xyz="0 0 0" rpy="${PI/2} 0 0"/>
-        <geometry>
-          <cylinder radius="0.07" length="0.16"/>
-        </geometry>
-      </collision>
-      <xacro:cylinder_inertial mass="0.7" radius="0.07" length="0.16"/>
-    </link>
-    <joint name="${name}_hub_joint" type="fixed">
-      <parent link="${name}_leg_link"/>
-      <child link="${name}_hub_link"/>
-      <origin xyz="0 0 ${-leg_length/2}" rpy="0 0 0"/>
-    </joint>
-    <link name="${name}_wheel_link">
-      <visual>
-        <origin xyz="0 0 0" rpy="${PI/2} 0 0"/>
-        <geometry>
-          <cylinder radius="${wheel_radius}" length="${wheel_width}"/>
-        </geometry>
-        <material name="rubber">
-          <color rgba="0.02 0.02 0.02 1.0"/>
-        </material>
-      </visual>
-      <collision>
-        <origin xyz="0 0 0" rpy="${PI/2} 0 0"/>
-        <geometry>
-          <cylinder radius="${wheel_radius}" length="${wheel_width}"/>
-        </geometry>
-      </collision>
-      <xacro:cylinder_inertial mass="2.4" radius="${wheel_radius}" length="${wheel_width}"/>
-    </link>
-    <joint name="${name}_wheel_joint" type="continuous">
-      <parent link="${name}_hub_link"/>
-      <child link="${name}_wheel_link"/>
-      <origin xyz="0 0 0" rpy="0 0 0"/>
-      <axis xyz="0 1 0"/>
-      <dynamics damping="0.20" friction="0.10"/>
-    </joint>
-    <transmission name="${name}_wheel_transmission">
-      <type>transmission_interface/SimpleTransmission</type>
-      <joint name="${name}_wheel_joint">
-        <hardwareInterface>velocity</hardwareInterface>
-      </joint>
-      <actuator name="${name}_wheel_motor">
-        <hardwareInterface>velocity</hardwareInterface>
-        <mechanicalReduction>1</mechanicalReduction>
-      </actuator>
-    </transmission>
-    <gazebo reference="${name}_leg_link">
-      <material>Gazebo/Grey</material>
-    </gazebo>
-    <gazebo reference="${name}_hub_link">
-      <material>Gazebo/Grey</material>
-    </gazebo>
-    <gazebo reference="${name}_wheel_link">
-      <material>Gazebo/Black</material>
-      <mu1>1.45</mu1>
-      <mu2>1.45</mu2>
-      <kp>1000000</kp>
-      <kd>1</kd>
-    </gazebo>
-  </xacro:macro>
-</robot>
+/home/sukru/ika_teknofest_aventra_ws/src/ika_description/urdf/wheels.xacro

File: src/ika_description/urdf/lidar.xacro (robot description, xacro)
@@ -1,17 +1,72 @@
 <?xml version="1.0"?>
 <robot xmlns:xacro="http://www.ros.org/wiki/xacro">
+  <!--
+    Gazebo/RViz uyumlu 2D LiDAR modeli.
+    Konum robot.urdf.xacro içindeki xacro:lidar_sensor çağrısından gelir;
+    bu dosyada x/y/z değerleri değiştirilmez.
+  -->
   <xacro:macro name="lidar_sensor" params="parent x y z">
+    <joint name="lidar_joint" type="fixed">
+      <parent link="${parent}"/>
+      <child link="lidar_link"/>
+      <origin xyz="${x} ${y} ${z}" rpy="0 0 0"/>
+    </joint>
     <link name="lidar_link">
-      <visual><geometry><cylinder radius="0.06" length="0.05"/></geometry><material name="black"><color rgba="0 0 0 1"/></material></visual>
-      <collision><geometry><cylinder radius="0.06" length="0.05"/></geometry></collision>
-      <inertial><mass value="0.25"/><inertia ixx="0.0003" ixy="0" ixz="0" iyy="0.0003" iyz="0" izz="0.0003"/></inertial>
+      <visual>
+        <geometry>
+          <cylinder radius="0.05" length="0.04"/>
+        </geometry>
+        <material name="black">
+          <color rgba="0 0 0 1"/>
+        </material>
+      </visual>
+      <visual>
+        <origin xyz="0 0 -0.05" rpy="0 0 0"/>
+        <geometry>
+          <cylinder radius="0.01" length="0.1"/>
+        </geometry>
+        <material name="black">
+          <color rgba="0 0 0 1"/>
+        </material>
+      </visual>
+      <collision>
+        <geometry>
+          <cylinder radius="0.05" length="0.04"/>
+        </geometry>
+      </collision>
+      <inertial>
+        <origin xyz="0 0 0" rpy="0 0 0"/>
+        <mass value="0.1"/>
+        <inertia
+          ixx="0.0000266667" ixy="0" ixz="0"
+          iyy="0.0000266667" iyz="0"
+          izz="0.000125"/>
+      </inertial>
     </link>
-    <joint name="lidar_joint" type="fixed"><parent link="${parent}"/><child link="lidar_link"/><origin xyz="${x} ${y} ${z}" rpy="0 0 0"/></joint>
     <gazebo reference="lidar_link">
-      <sensor name="lidar" type="ray">
+      <material>Gazebo/Black</material>
+      <sensor name="laser" type="ray">
+        <pose>0 0 0 0 0 0</pose>
+        <visualize>false</visualize>
         <update_rate>10</update_rate>
-        <ray><scan><horizontal><samples>720</samples><resolution>1</resolution><min_angle>-3.14159</min_angle><max_angle>3.14159</max_angle></horizontal></scan><range><min>0.12</min><max>12.0</max><resolution>0.01</resolution></range></ray>
-        <plugin name="lidar_controller" filename="libgazebo_ros_ray_sensor.so">
-          <ros><remapping>~/out:=scan</remapping></ros>
+        <ray>
+          <scan>
+            <horizontal>
+              <samples>360</samples>
+              <resolution>1</resolution>
+              <min_angle>-3.14</min_angle>
+              <max_angle>3.14</max_angle>
+            </horizontal>
+          </scan>
+          <range>
+            <min>0.3</min>
+            <max>12</max>
+            <resolution>0.01</resolution>
+          </range>
+        </ray>
+        <plugin name="laser_controller" filename="libgazebo_ros_ray_sensor.so">
+          <ros>
+            <argument>~/out:=scan</argument>
+          </ros>
           <output_type>sensor_msgs/LaserScan</output_type>
           <frame_name>lidar_link</frame_name>

File: src/ika_description/urdf/robot.urdf.xacro (robot description, xacro)
@@ -2,4 +2,7 @@
 <robot name="ika_teknofest_aventra" xmlns:xacro="http://www.ros.org/wiki/xacro">
   <xacro:property name="PI" value="3.14159265359"/>
+  <!-- TEKNOFEST UPDATE: ornek projedeki gibi robot modeli launch argumanlariyla yonetilebilir hale getirildi. -->
+  <xacro:arg name="use_ros2_control" default="true"/>
+  <xacro:arg name="sim_mode" default="false"/>
   <!-- Gerçek rapora yakın genel boyutlar: 1.40 m uzunluk, 0.95 m genişlik. -->
   <xacro:property name="base_length" value="1.40"/>
@@ -25,4 +28,7 @@
   <xacro:include filename="$(find ika_description)/urdf/environmental_sensor.xacro"/>
   <xacro:include filename="$(find ika_description)/urdf/laser_pointer.xacro"/>
+  <!-- TEKNOFEST UPDATE: kontrol bloklari ayri xacro dosyalarina bolundu. -->
+  <xacro:include filename="$(find ika_description)/urdf/ros2_control.xacro"/>
+  <xacro:include filename="$(find ika_description)/urdf/gazebo_control.xacro"/>
   <!-- Ana gövde ve üst sensör şasesi -->
   <xacro:ika_base/>
@@ -45,34 +51,12 @@
   <xacro:laser_pointer parent="sensor_deck_link" x="0.28" y="0.00" z="0.16"/>
   <xacro:aim_camera parent="tilt_link" x="0.12" y="0.00" z="0.03" roll="0" pitch="0" yaw="0"/>
-    <!-- gazebo_ros2_control plugin -->
-  <gazebo>
-    <plugin name="gazebo_ros2_control" filename="libgazebo_ros2_control.so">
-      <parameters>$(arg controllers_file)</parameters>
-    </plugin>
-  </gazebo>
-  <ros2_control name="ika_hw" type="system">
-    <hardware>
-      <plugin>gazebo_ros2_control/GazeboSystem</plugin>
-    </hardware>
-    <joint name="front_left_wheel_joint">
-      <command_interface name="velocity"/>
-      <state_interface name="position"/>
-      <state_interface name="velocity"/>
-    </joint>
-    <joint name="rear_left_wheel_joint">
-      <command_interface name="velocity"/>
-      <state_interface name="position"/>
-      <state_interface name="velocity"/>
-    </joint>
-    <joint name="front_right_wheel_joint">
-      <command_interface name="velocity"/>
-      <state_interface name="position"/>
-      <state_interface name="velocity"/>
-    </joint>
-    <joint name="rear_right_wheel_joint">
-      <command_interface name="velocity"/>
-      <state_interface name="position"/>
-      <state_interface name="velocity"/>
-    </joint>
-  </ros2_control>
+  <!-- TEKNOFEST UPDATE: Ornek projedeki kosullu kontrol secimi Teknofest robotuna eklendi.
+       use_ros2_control:=true -> gazebo_ros2_control + controller_manager
+       use_ros2_control:=false -> basit Gazebo diff_drive fallback -->
+  <xacro:if value="$(arg use_ros2_control)">
+    <xacro:ika_ros2_control controllers_file="$(arg controllers_file)"/>
+  </xacro:if>
+  <xacro:unless value="$(arg use_ros2_control)">
+    <xacro:ika_gazebo_diff_drive/>
+  </xacro:unless>
 </robot>
